File: hackpad.kicad_pcb (KiCad board)
At the start: 2 copper layers, 59 x 99 mm, 24 parts, among them SW1 SW_Push, SW10 SW_Push, SW12 SW_Push, SW2 SW_Push, SW3 SW_Push, SW4 SW_Push, SW5 SW_Push, SW6 SW_Push, SW7 SW_Push, SW8 RotaryEncoder_Switch, SW9 SW_Push, U1 XIAO-RP2040-DIP

Commit message: h
Other:
- board text added: "XIAO HERE!"
- board text added: "jonathan.. pad"
